File: electric/schematic/codec_sheet.sch (KiCad schematic (older format))
At the start: 7 parts

Commit message: Connected CODEC
Parts:
- added C? (x3): 0.1uF, symbol C
- added C? (x5): 1uF, symbol C
- added R? (x10): R0R, symbol R
Connections:
- net CODEC_I2C_SCL: now also U?.9 (SCL/nSS)
- net CODEC_I2C_SDA: now also U?.10 (SDA/MOSI)
- net CODEC_I2S_CLK: now also U?.2 (BCLK), R?.1
- net CODEC_I2S_DIN: now also U?.4 (DIN/MFP1)
- net CODEC_I2S_DOUT: now also U?.5 (DOUT/MFP2)
- net CODEC_I2S_FSYNC: now also U?.3 (WCLK)
- net at U?.1 (MCLK): now also R?.2
- net at U?.11 (MISO/MFP4): now also R?.1
- net at U?.12 (SPI_SELECT): now also R?.1
- net at U?.17 (AVss): now also R?.1
- net at U?.18 (REF): now also C?.1
- net at U?.24 (AVdd): now also R?.1
- net CODEC_3V3: now reaches U?.26 (LDOIN)
- net CODEC_3V3: now also U?.6 (IOVdd), C?.1, C?.1, C?.1, C?.1, R?.1
- net at U?.28 (DVss): now also R?.2
- net at U?.29 (DVdd): now also C?.1
- net at U?.30 (LDO_SELECT): now also C?.2, C?.2, R?.2
- net #CODEC_RESET: now reaches U?.31 (nRESET)
- net #CODEC_RESET: now also R?.1
- net at U?.32 (GPIO_MFP5): now also R?.2
- net GND: now reaches U?.33 (PAD_GND)
- net GND: now also U?.7 (IOVss), C?.1, C?.1, C?.2, C?.2, C?.2, C?.2, C?.2, C?.2, R?.1, R?.1, R?.2, R?.2, R?.2, R?.2
- net at U?.8 (SCLK/MFP3): now also R?.1
- new net CODEC_AVDD: R?.2
- new net RADIO_GPIO6: R?.2
Other:
- moved on the sheet: R?, U?

Commit message: Class D amplifier
Parts:
- added C? (x2): 4.7nF, symbol C
- added C? (x4): 0.1uF, symbol C
- added R? (x4): 1K, symbol R
- added R? (x10): R0R, symbol R
- added U?: TPA2012, symbol TPA2012
Connections:
- net GND: now also R?.1, R?.1, R?.1, R?.2, R?.2, R?.2
- net CCODEC_LOL: now reaches U?.22 (LOL)
- net CCODEC_LOL: now also R?.1
- net CCODEC_LOR: now reaches U?.23 (LOR)
- net CCODEC_LOR: now also R?.1
- new net: R?.2, U?.12 (PGND)
- new net: R?.2, U?.13 (PVDD)
- new net: R?.1, U?.18 (AGND)
- new net: R?.1, U?.3 (PVDD)
- new net: R?.1, U?.4 (PGND)
- new net: R?.1, U?.~ (T_PAD)
- new net: C?.1, C?.2, R?.2 (x2)
- new net: C?.2, C?.2, R?.2 (x2)
- new net AMPLY_GAIN0: R?.2, U?.15 (G0)
- new net AMPLY_GAIN1: R?.2, U?.1 (G1)
- new net AMPLY_L+: C?.1, U?.20 (INL+)
- new net AMPLY_L-: C?.1, U?.19 (INL-)
- new net AMPLY_LOUT+: U?.2 (OUTL+)
- new net AMPLY_LOUT-: U?.5 (OUTL-)
- new net AMPLY_R+: C?.1, U?.16 (INR+)
- new net AMPLY_R-: C?.1, U?.17 (INR-)
- new net AMPLY_ROUT+: U?.14 (OUTR+)
- new net AMPLY_ROUT-: U?.11 (OUTR-)
- new net AMPLY_VDD: R?.1, R?.2
- new net RADIO_GPIO2: R?.1
- new net RADIO_GPIO3: R?.1
- new net RADIO_GPIO4: R?.1
- new net RADIO_GPIO5: R?.1
- new net SHUT_DOWN_L: R?.2, U?.7 (#SDL)
- new net SHUT_DOWN_R: R?.2, U?.8 (#SDR)
- no-connect marks 0 -> 2
Other:
- moved on the sheet: R?

Commit message: Some notes
Other:
- note added: "Missed: \npower amplifier, \npower codec,\nmicrophone\n"
Changed lines of the file:
@@
 Text GLabel 6100 7900 2    60   Input ~ 0
 AMPLY_R+
+Text Notes 8350 8450 0    197  ~ 0
+Missed: \npower amplifier, \npower codec,\nmicrophone\n
 $EndSCHEMATC
