File: electric/schematic/radio_sheet.sch (KiCad schematic (older format))
At the start: 348 parts

Commit message: Connected CODEC
Connections:
- net RADIO_GPIO6: now reaches U?.61 (GPIO6)
Changed lines of the file:
@@
 Text GLabel 13850 4450 2    60   BiDi ~ 0
 RADIO_I2S_CLK
+Text GLabel 7650 4950 2    60   Input ~ 0
+RADIO_GPIO6
+Wire Wire Line
+	7500 4950 7650 4950
 $EndSCHEMATC

Commit message: Class D amplifier
Connections:
- net RADIO_GPIO2: now reaches U?.57 (GPIO2)
- net RADIO_GPIO3: now reaches U?.58 (GPIO3)
- net RADIO_GPIO4: now reaches U?.59 (GPIO4)
- net RADIO_GPIO5: now reaches U?.60 (GPIO5)
Changed lines of the file:
@@
 Wire Wire Line
 	7500 4950 7650 4950
+Text GLabel 7650 4850 2    60   Input ~ 0
+RADIO_GPIO5
+Text GLabel 7650 4750 2    60   Input ~ 0
+RADIO_GPIO4
+Text GLabel 7650 4650 2    60   Input ~ 0
+RADIO_GPIO3
+Text GLabel 7650 4550 2    60   Input ~ 0
+RADIO_GPIO2
+Wire Wire Line
+	7650 4550 7500 4550
+Wire Wire Line
+	7500 4650 7650 4650
+Wire Wire Line
+	7650 4750 7500 4750
+Wire Wire Line
+	7500 4850 7650 4850
 $EndSCHEMATC

Commit message: Touch part started
Parts:
- removed C? (x39): 0.1uF, symbol C
- removed C? (x9): 4.7uF, symbol C
- removed C? (x9): 10uF, symbol C
- removed C? (x6): 22uF, symbol C
- removed C? (x3): 0.5pF, symbol C
- removed FL? (x3): Band_pass_filter, symbol Band_pass_filter
- removed J? (x3): Conn_02x03_Counter_Clockwise, symbol Conn_02x03_Counter_Clockwise
- removed J? (x3): Conn_02x07_Odd_Even, symbol Conn_02x07_Odd_Even
- removed L? (x6): 2.2uH, symbol L
- removed L? (x3): 1uH, symbol L
- removed L? (x3): 10uH, symbol L
- removed L? (x3): 3.3uH, symbol L
- removed R? (x87): R0R, symbol R
- removed R? (x3): 2.7K, symbol R
- removed R? (x6): 100K, symbol R
- removed R? (x3): 270R, symbol R
- removed R? (x3): 10K, symbol R
- removed TP? (x57): TEST, symbol TEST
- removed U? (x3): CC3220SF, symbol CC3220SF
- removed U? (x3): AH316M245001-T, symbol AH316M245001-T
- removed U? (x3): MX25R3235FM1IL0, symbol MX25R3235FM1IL0
- removed Y? (x3): 40 MHz, symbol Crystal_GND24
Connections:
- net GND: no longer R?.1, R?.1, R?.1, R?.1, R?.1, R?.2, R?.2
- net I2C_SCL_R: no longer R?.2, R?.2, R?.2, R?.2, R?.2, U?.2 (GPIO11), U?.50 (GPIO0), U?.53 (GPIO30), U?.63 (GPIO8), U?.64 (GPIO9)
- net RADIO_I2C_SCL: no longer R?.1
- net RADIO_I2C_SDA: no longer R?.1
- new net I2C_SDA_R: R?.2, U?.2 (GPIO11)
- new net I2S_CLK_R: R?.2, U?.53 (GPIO30)
- new net I2S_DIN_R: R?.2, U?.50 (GPIO0)
- new net I2S_DOUT_R: R?.2, U?.64 (GPIO9)
- new net I2S_FSYNC_R: R?.2, U?.63 (GPIO8)
- new net RADIO_I2S_DIN: R?.1
- new net RADIO_I2S_FSYNC: R?.1
- new net Radio_VCC: R?.1, R?.1, R?.1, R?.1, R?.1, R?.2, R?.2
- no-connect marks 12 -> 3
